File: LogicGates.kicad_pcb (KiCad board)
At the start: 2 copper layers, 12 parts, among them Q1 2N3904, Q2 2N3904, Q3 2N3906, SW1 SW_DIP_x02

Commit message: Add files via upload
Parts:
- added D2: LED, LED_SMD:LED_0402_1005Metric, F.Cu at (81.3, 38.3)
- added D3: LED, LED_SMD:LED_0402_1005Metric, F.Cu at (81.3, 40.3)
- added D4: LED, LED_SMD:LED_0402_1005Metric, F.Cu at (81.3, 42.3)
- added D5: LED, LED_SMD:LED_0402_1005Metric, F.Cu at (132.2, 53.5)
- added D6: LED, LED_SMD:LED_0402_1005Metric, F.Cu at (133.7, 65.4)
- added D7: LED, LED_SMD:LED_0402_1005Metric, F.Cu at (81.3, 48.3)
- added Q10: 2N3904, Package_TO_SOT_THT:TO-92_Inline, F.Cu at (128.8, 68.9)
- added Q11: 2N3904, Package_TO_SOT_THT:TO-92_Inline, F.Cu at (68.6, 50.2)
- added Q12: 2N3904, Package_TO_SOT_THT:TO-92_Inline, F.Cu at (68.6, 56.0)
- added Q13: 2N3904, Package_TO_SOT_THT:TO-92_Inline, F.Cu at (75.1, 38.6)
- added Q14: 2N3904, Package_TO_SOT_THT:TO-92_Inline, F.Cu at (75.1, 44.4)
- added Q15: 2N3904, Package_TO_SOT_THT:TO-92_Inline, F.Cu at (75.1, 50.2)
- added Q16: 2N3904, Package_TO_SOT_THT:TO-92_Inline, F.Cu at (75.1, 56.0)
- added Q4: 2N3904, Package_TO_SOT_THT:TO-92_Inline, F.Cu at (55.6, 56.0)
- added Q5: 2N3904, Package_TO_SOT_THT:TO-92_Inline, F.Cu at (62.1, 38.6)
- added Q6: 2N3904, Package_TO_SOT_THT:TO-92_Inline, F.Cu at (62.1, 44.4)
- added Q7: 2N3904, Package_TO_SOT_THT:TO-92_Inline, F.Cu at (128.8, 57.9)
- added Q8: 2N3904, Package_TO_SOT_THT:TO-92_Inline, F.Cu at (128.8, 63.4)
- added Q9: 2N3904, Package_TO_SOT_THT:TO-92_Inline, F.Cu at (132.3, 68.6)
- added R10: 1k, Resistor_SMD:R_0402_1005Metric, F.Cu at (70.6, 65.5)
- added R11: 330R, Resistor_SMD:R_0402_1005Metric, F.Cu at (70.6, 67.5)
- added R12: 330R, Resistor_SMD:R_0402_1005Metric, F.Cu at (70.6, 69.4)
- added R13: 330R, Resistor_SMD:R_0402_1005Metric, F.Cu at (130.3, 53.5)
- added R14: 1k, Resistor_SMD:R_0402_1005Metric, F.Cu at (128.8, 52.0)
- added R15: 330R, Resistor_SMD:R_0402_1005Metric, F.Cu at (131.8, 65.4)
- added R16: 1k, Resistor_SMD:R_0402_1005Metric, F.Cu at (131.3, 64.0)
- added R17: 1k, Resistor_SMD:R_0402_1005Metric, F.Cu at (73.5, 67.5)
- added R18: 1k, Resistor_SMD:R_0402_1005Metric, F.Cu at (73.5, 69.4)
- added R19: 10k, Resistor_SMD:R_0402_1005Metric, F.Cu at (76.4, 59.5)
- added R20: 1k, Resistor_SMD:R_0402_1005Metric, F.Cu at (76.4, 61.5)
- added R21: 330R, Resistor_SMD:R_0402_1005Metric, F.Cu at (76.4, 63.5)
- added R22: 1k, Resistor_SMD:R_0402_1005Metric, F.Cu at (119.6, 52.1)
- added R23: 1k, Resistor_SMD:R_0402_1005Metric, F.Cu at (117.4, 52.1)
- added R7: 330R, Resistor_SMD:R_0402_1005Metric, F.Cu at (70.6, 59.5)
- added R8: 1k, Resistor_SMD:R_0402_1005Metric, F.Cu at (70.6, 61.5)
- added R9: 330R, Resistor_SMD:R_0402_1005Metric, F.Cu at (70.6, 63.5)
- Q3: value 2N3906 -> 2N3904
- moved R3 60.8 mm to (121.5, 52.1), turned to 180 degrees
- moved R4 55.1 mm to (115.5, 52.1)
- moved U1 54.2 mm to (118.5, 36.1)
- moved R2 53.8 mm to (124.3, 33.3), turned to -90 degrees
- moved R1 42.6 mm to (112.7, 33.3), turned to -90 degrees
- moved SW1 37.9 mm to (118.5, 45.8), turned to -90 degrees
- moved D1 29.0 mm to (81.3, 36.3), turned to 0 degrees
- moved R5 8.80 mm to (67.7, 67.5)
- moved R6 8.80 mm to (67.7, 69.4)
- moved Q1 7.96 mm to (55.6, 38.6)
- moved Q2 7.96 mm to (55.6, 44.4)
- moved Q3 7.86 mm to (55.6, 50.2)
Connections:
- D1 pad 1: GND -> Net-(D1-K)
- Q1 pad 1: Net-(Q1-E) -> GND
- Q1 pad 3: +5V -> Net-(D1-A)
- Q2 pad 1: Net-(D1-A) -> GND
- Q2 pad 3: Net-(Q1-E) -> Net-(D2-A)
- Q3 pad 1: unconnected-(Q3-E-Pad1) -> Net-(Q3-E)
- Q3 pad 2: unconnected-(Q3-B-Pad2) -> A
- Q3 pad 3: unconnected-(Q3-C-Pad3) -> +5V
- R3 pad 2: Net-(R3-Pad2) -> Net-(R22-Pad2)
- R4 pad 2: Net-(R4-Pad2) -> Net-(R23-Pad2)
- R5 pad 1: A -> +5V
- R5 pad 2: Net-(R3-Pad2) -> Net-(Q11-C)
- R6 pad 1: B -> Net-(Q14-B)
- R6 pad 2: Net-(R4-Pad2) -> Net-(Q11-C)
- SW1 pad 3: Net-(R4-Pad2) -> Net-(R23-Pad2)
- SW1 pad 4: Net-(R3-Pad2) -> Net-(R22-Pad2)
Routing:
- net +5V: track 4.49 -> 57.8 mm
- net GND: track 0.00 -> 52.4 mm, vias 0 -> 4
- net A: track 0.00 -> 45.5 mm
- net B: track 0.00 -> 33.1 mm, vias 0 -> 2
- net Net-(Q10-C): track 0.00 -> 11.0 mm
- net Net-(U1-CC1): track 0.00 -> 6.62 mm
- net Net-(U1-CC2): track 0.00 -> 6.61 mm
- net Net-(Q7-C): track 0.00 -> 4.01 mm
- net Net-(Q7-E): track 0.00 -> 2.96 mm
- net Net-(R22-Pad2): track 0.00 -> 2.95 mm
- net Net-(R23-Pad2): track 0.00 -> 2.94 mm
- net Net-(D5-A): track 0.00 -> 0.91 mm
- net Net-(D6-A): track 0.00 -> 0.90 mm
- added copper zone on B.Cu, net GND
Other:
- board text added: "NAND Gate"
- board text added: "NOR Gate"

Commit message: Add files via upload
Parts:
- R20, R22, R23, R6: value 1k -> 10k
- moved D5 10.6 mm to (142.8, 53.6)
- moved R16 9.70 mm to (139.6, 58.8)
Connections:
- Q13 pad 3: Net-(Q13-C) -> +5V
- Q14 pad 1: GND -> Net-(Q14-E)
- R17 pad 1: +5V -> Net-(Q14-E)
- R17 pad 2: Net-(Q13-C) -> GND
- R21 pad 1: GND -> Net-(Q14-E)
Routing:
- net +5V: track 57.8 -> 39.1 mm
- net GND: track 52.4 -> 40.9 mm, vias 4 -> 3
Other:
- board text removed: "NAND Gate"
- board text removed: "NOR Gate"
Changed lines of the file:
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@@
 	(net 22 "Net-(Q11-E)")
 	(net 23 "Net-(Q11-C)")
-	(net 24 "Net-(Q13-C)")
+	(net 24 "Net-(Q14-E)")
 	(net 25 "Net-(Q13-E)")
 	(net 26 "Net-(Q13-B)")
@@
 			)
 		)
-		(property "Value" "1k"
+		(property "Value" "10k"
 			(at 0 1.17 0)
 			(layer "F.Fab")
@@
 	(footprint "LED_SMD:LED_0402_1005Metric"
 		(layer "F.Cu")
-		(at 132.2 53.45 180)
+		(at 142.7825 53.6 180)
 		(descr "LED SMD 0402 (1005 Metric), square (rectangular) end terminal, IPC-7351 nominal, (Body size source: http://www.tortai-tech.com/upload/download/2011102023233369053.pdf), generated with kicad-footprint-generator")
 		(tags "LED")
@@
 			)
 		)
-		(property "Value" "1k"
+		(property "Value" "10k"
 			(at 0 1.17 0)
 			(layer "F.Fab")
@@
 			(layers "*.Cu" "*.Mask")
 			(remove_unused_layers no)
-			(net 24 "Net-(Q13-C)")
+			(net 8 "+5V")
 			(pinfunction "C")
 			(pintype "passive")
@@
 			(layers "F.Cu" "F.Mask" "F.Paste")
 			(roundrect_rratio 0.25)
-			(net 8 "+5V")
+			(net 24 "Net-(Q14-E)")
 			(pintype "passive")
 		)
@@
 			(layers "F.Cu" "F.Mask" "F.Paste")
 			(roundrect_rratio 0.25)
-			(net 24 "Net-(Q13-C)")
+			(net 9 "GND")
 			(pintype "passive")
 		)
@@
 	(footprint "Resistor_SMD:R_0402_1005Metric"
 		(layer "F.Cu")
-		(at 131.35 63.99 -90)
+		(at 139.55 58.81 -90)
 		(descr "Resistor SMD 0402 (1005 Metric), square (rectangular) end terminal, IPC-7351 nominal, (Body size source: IPC-SM-782 page 72, https://www.pcb-3d.com/wordpress/wp-content/uploads/ipc-sm-782a_amendment_1_and_2.pdf), generated with kicad-footprint-generator")
 		(tags "resistor")
@@
 			(layers "*.Cu" "*.Mask")
 			(remove_unused_layers no)
-			(net 9 "GND")
+			(net 24 "Net-(Q14-E)")
 			(pinfunction "E")
 			(pintype "passive")
@@
 			)
 		)
-		(property "Value" "1k"
+		(property "Value" "10k"
 			(at 0 1.17 0)
 			(layer "F.Fab")
@@
 			(layers "F.Cu" "F.Mask" "F.Paste")
 			(roundrect_rratio 0.25)
-			(net 9 "GND")
+			(net 24 "Net-(Q14-E)")
 			(pintype "passive")
 		)
@@
 			)
 		)
-		(property "Value" "1k"
+		(property "Value" "10k"
 			(at 0 1.17 0)
 			(layer "F.Fab")
@@
 			(remove_unused_layers no)
 			(net 9 "GND")
-			(pinfunction "MH1")
+			(pinfunction "MH3")
 			(pintype "input")
 		)
@@
 			(remove_unused_layers no)
 			(net 9 "GND")
-			(pinfunction "MH1")
+			(pinfunction "MH3")
 			(pintype "input")
 		)
@@
 			(remove_unused_layers no)
 			(net 9 "GND")
-			(pinfunction "MH1")
+			(pinfunction "MH3")
 			(pintype "input")
 		)
@@
 			(remove_unused_layers no)
 			(net 9 "GND")
-			(pinfunction "MH1")
+			(pinfunction "MH3")
 			(pintype "input")
 		)
@@
 		)
 	)
-	(gr_text "NOR Gate"
-		(at 136.25 65.9 90)
-		(layer "F.SilkS")
-		(effects
-			(font
-				(size 1 1)
-				(thickness 0.1)
-			)
-			(justify left bottom)
-		)
-	)
-	(gr_text "NAND Gate"
-		(at 129.65 52.8 0)
-		(layer "F.SilkS")
-		(effects
-			(font
-				(size 1 1)
-				(thickness 0.1)
-			)
-			(justify left bottom)
-		)
-	)
 	(segment
 		(start 133.6 67.89)
@@
 	(segment
 		(start 128.85 47.55)
-		(end 133.45 52.15)
-		(width 0.5)
-		(layer "F.Cu")
-		(net 8)
-	)
-	(segment
-		(start 128.85 47.55)
 		(end 128.85 51.53)
 		(width 0.5)
@@
 	)
 	(segment
-		(start 133.45 52.15)
-		(end 133.45 60.65)
-		(width 0.5)
-		(layer "F.Cu")
-		(net 8)
-	)
-	(segment
-		(start 131.35 63.48)
-		(end 131.35 62.75)
-		(width 0.5)
-		(layer "F.Cu")
-		(net 8)
-	)
-	(segment
 		(start 116.98 32.97)
 		(end 116.98 32.511986)
@@
 	)
 	(segment
-		(start 131.35 62.75)
-		(end 133.45 60.65)
-		(width 0.5)
-		(layer "F.Cu")
-		(net 8)
-	)
-	(segment
 		(start 113.48 33.85)
 		(end 114.18 33.15)
@@
 	)
 	(segment
-		(start 129.075 63.44)
-		(end 132.685 59.83)
-		(width 0.2)
-		(layer "F.Cu")
-		(net 9)
-	)
-	(segment
 		(start 132.33 68.61)
 		(end 132.33 67.24)
@@
 	)
 	(segment
-		(start 132.685 59.83)
-		(end 132.685 53.45)
-		(width 0.2)
-		(layer "F.Cu")
-		(net 9)
-	)
-	(segment
 		(start 123.49 33.82)
 		(end 122.82 33.15)
@@
 		(size 0.6)
 		(drill 0.3)
-		(layers "F.Cu" "B.Cu")
-		(net 9)
-	)
-	(via
-		(at 132.685 59.83)
-		(size 0.6)
-		(drill 0.3)

Commit message: Add files via upload
Parts:
- removed Q16: 2N3904, Package_TO_SOT_THT:TO-92_Inline
- removed R18: 1k, Resistor_SMD:R_0402_1005Metric
- removed R20, R6: 10k, Resistor_SMD:R_0402_1005Metric
- moved Q3 75.0 mm to (127.4, 71.9), turned to -90 degrees
- moved Q4 72.6 mm to (127.4, 66.4), turned to -90 degrees
- moved Q5 71.0 mm to (123.3, 74.4), turned to 90 degrees
- moved Q6 66.0 mm to (123.3, 68.9), turned to 90 degrees
- moved Q1 60.5 mm to (113.7, 55.4), turned to -90 degrees
- moved Q2 60.4 mm to (113.7, 60.9), turned to -90 degrees
- moved D3 58.8 mm to (125.9, 78.7), turned to 90 degrees
- moved R7 57.9 mm to (125.9, 76.8), turned to -90 degrees
- moved D4 56.8 mm to (124.9, 78.7), turned to 90 degrees
- moved R12 54.8 mm to (124.9, 76.8), turned to -90 degrees
- moved D1 52.6 mm to (115.0, 76.8), turned to 90 degrees
- moved D2 49.9 mm to (113.1, 76.8), turned to 90 degrees
- moved Q14 47.4 mm to (113.7, 71.8), turned to -90 degrees
- moved Q12 46.3 mm to (113.7, 66.4), turned to -90 degrees
- moved R9 45.4 mm to (114.0, 76.8), turned to -90 degrees
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Connections:
- Q14 pad 2: Net-(Q14-B) -> B
- Q15 pad 1: Net-(Q15-E) -> Net-(Q14-E)
- Q15 pad 3: Net-(Q15-C) -> Net-(Q13-E)
- R19 pad 1: Net-(Q15-E) -> Net-(Q13-B)
- R19 pad 2: GND -> Net-(Q11-C)
Routing:
- net +5V: track 39.1 -> 104.9 mm, vias 0 -> 1
- net Net-(D2-A): track 0.00 -> 29.7 mm
- net Net-(D1-A): track 0.00 -> 27.4 mm
- net Net-(Q7-C): track 4.01 -> 26.0 mm, vias 0 -> 1
- net B: track 33.1 -> 54.4 mm
- net A: track 45.5 -> 66.1 mm, vias 0 -> 4
- net Net-(Q10-C): track 11.0 -> 27.6 mm
- net Net-(Q11-C): track 0.00 -> 16.4 mm
- net GND: track 40.9 -> 56.3 mm
- net Net-(Q13-E): track 0.00 -> 14.4 mm
- net Net-(Q4-E): track 0.00 -> 13.1 mm
- net Net-(Q14-E): track 0.00 -> 11.2 mm
- net Net-(Q5-E): track 0.00 -> 9.21 mm
- net Net-(Q11-E): track 0.00 -> 4.03 mm
- net Net-(Q13-B): track 0.00 -> 3.87 mm
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Other:
- board outline added: 27 x 50 mm
- board text added: "AND"
- board text added: "NAND"
- board text added: "NOR"
- board text added: "NOT A"
- board text added: "NOT B"
- board text added: "OR"
- board text added: "XOR"
