File: LogicGates.kicad_sch (KiCad schematic)
At the start: 48 parts, among them Q1 2N3904, Q10 2N3904, Q11 2N3904, Q12 2N3904, Q13 2N3904, Q14 2N3904, Q15 2N3904, Q16 2N3904, Q2 2N3904, Q3 2N3904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

Commit message: Add files via upload
Parts:
- R20, R22, R23, R6: value 1k -> 10k
Connections:
- net +5V: now also Q13.3 (C); no longer R17.1
- net GND: now also R17.2; no longer Q14.1 (E), R21.1
- new net: Q14.1 (E), R17.1, R21.1
Other:
- moved on the sheet: R17
Changed lines of the file:
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@@
 	)
 	(junction
-		(at 186.69 105.41)
+		(at 210.82 132.08)
 		(diameter 0)
 		(color 0 0 0 0)
 	)
 	(junction
-		(at 90.17 93.98)
+		(at 186.69 105.41)
 		(diameter 0)
 		(color 0 0 0 0)
 	)
 	(junction
-		(at 86.36 41.91)
+		(at 90.17 93.98)
 		(diameter 0)
 		(color 0 0 0 0)
 	)
 	(junction
-		(at 210.82 132.08)
+		(at 86.36 41.91)
 		(diameter 0)
 		(color 0 0 0 0)
@@
 	(wire
 		(pts
-			(xy 210.82 90.17) (xy 210.82 91.44)
+			(xy 210.82 132.08) (xy 210.82 133.35)
 		)
 		(stroke
@@
 	(wire
 		(pts
-			(xy 210.82 132.08) (xy 210.82 133.35)
-		)
-		(stroke
-			(width 0)
-			(type default)
-		)
-	)
-	(wire
-		(pts
 			(xy 66.04 71.12) (xy 69.85 71.12)
 		)
@@
 	(wire
 		(pts
-			(xy 210.82 99.06) (xy 210.82 100.33)
-		)
-		(stroke
-			(width 0)
-			(type default)
-		)
-	)
-	(wire
-		(pts
 			(xy 90.17 111.76) (xy 90.17 113.03)
 		)
@@
 	(wire
 		(pts
+			(xy 210.82 97.79) (xy 210.82 100.33)
+		)
+		(stroke
+			(width 0)
+			(type default)
+		)
+	)
+	(wire
+		(pts
 			(xy 125.73 38.1) (xy 128.27 38.1)
 		)
@@
 	(wire
 		(pts
+			(xy 210.82 140.97) (xy 210.82 142.24)
+		)
+		(stroke
+			(width 0)
+			(type default)
+		)
+	)
+	(wire
+		(pts
 			(xy 86.36 41.91) (xy 86.36 44.45)
 		)
@@
 	(symbol
 		(lib_id "Device:R")
-		(at 210.82 95.25 0)
+		(at 210.82 137.16 0)
 		(unit 1)
 		(exclude_from_sim no)
@@
 		(dnp no)
 		(property "Reference" "R17"
-			(at 213.36 95.25 90)
+			(at 213.36 137.16 90)
 			(effects
 				(font
@@
 		)
 		(property "Value" "1k"
-			(at 208.28 95.25 90)
+			(at 208.28 137.16 90)
 			(effects
 				(font
@@
 		)
 		(property "Footprint" "Resistor_SMD:R_0402_1005Metric"
-			(at 209.042 95.25 90)
+			(at 209.042 137.16 90)
 			(effects
 				(font
@@
 		)
 		(property "Datasheet" "~"
-			(at 210.82 95.25 0)
+			(at 210.82 137.16 0)
 			(effects
 				(font
@@
 		)
 		(property "Description" "Resistor"
-			(at 210.82 95.25 0)
+			(at 210.82 137.16 0)
 			(effects
 				(font
@@
 			)
 		)
-		(property "Value" "1k"
+		(property "Value" "10k"
 			(at 73.66 73.406 90)
 			(effects
@@
 			)
 		)
-		(property "Value" "1k"
+		(property "Value" "10k"
 			(at 195.58 107.95 90)
 			(effects
@@
 	(symbol
 		(lib_id "power:GND")
-		(at 210.82 133.35 0)
+		(at 210.82 142.24 0)
 		(unit 1)
 		(exclude_from_sim no)
@@
 		(fields_autoplaced yes)
 		(property "Reference" "#PWR022"
-			(at 210.82 139.7 0)
+			(at 210.82 148.59 0)
 			(effects
 				(font
@@
 		)
 		(property "Value" "GND"
-			(at 210.82 138.43 0)
+			(at 210.82 147.32 0)
 			(effects
 				(font
@@
 		)
 		(property "Footprint" ""
-			(at 210.82 133.35 0)
+			(at 210.82 142.24 0)
 			(effects
 				(font
@@
 		)
 		(property "Datasheet" ""
-			(at 210.82 133.35 0)
+			(at 210.82 142.24 0)
 			(effects
 				(font
@@
 		)
 		(property "Description" "Power symbol creates a global label with name \"GND\" , ground"
-			(at 210.82 133.35 0)
+			(at 210.82 142.24 0)
 			(effects
 				(font
@@
 			)
 		)
-		(property "Value" "1k"
+		(property "Value" "10k"
 			(at 73.66 66.04 90)
 			(effects
@@
 	(symbol
 		(lib_id "power:+5V")
-		(at 210.82 90.17 0)
+		(at 210.82 97.79 0)
 		(unit 1)
 		(exclude_from_sim no)
@@
 		(fields_autoplaced yes)
 		(property "Reference" "#PWR023"
-			(at 210.82 93.98 0)
+			(at 210.82 101.6 0)
 			(effects
 				(font
@@
 		)
 		(property "Value" "+5V"
-			(at 210.82 85.09 0)
+			(at 210.82 92.71 0)
 			(effects
 				(font
@@
 		)
 		(property "Footprint" ""
-			(at 210.82 90.17 0)
+			(at 210.82 97.79 0)
 			(effects
 				(font
@@
 		)
 		(property "Datasheet" ""
-			(at 210.82 90.17 0)
+			(at 210.82 97.79 0)
 			(effects
 				(font
@@
 		)
 		(property "Description" "Power symbol creates a global label with name \"+5V\""
-			(at 210.82 90.17 0)
+			(at 210.82 97.79 0)
 			(effects
 				(font
@@
 			)
 		)
-		(property "Value" "1k"
+		(property "Value" "10k"
 			(at 196.85 123.19 90)
 			(effects

Commit message: Add files via upload
Parts:
- removed Q16: 2N3904, Package_TO_SOT_THT:TO-92_Inline, symbol Transistor_BJT:2N3904
- removed R18: 1k, Resistor_SMD:R_0402_1005Metric, symbol Device:R
- removed R20, R6: 10k, Resistor_SMD:R_0402_1005Metric, symbol Device:R
Connections:
- net B: now also Q14.2 (B)
- net GND: no longer R19.2
- net at Q15.1 (E): now also Q14.1 (E), R17.1, R21.1; no longer R19.1
- net at Q15.3 (C): now also Q13.1 (E), Q14.3 (C)
- net at Q13.2 (B): now also R19.1
- net at Q11.3 (C), R5.2: now also R19.2
Other:
- moved on the sheet: D7, Q11, Q12, Q13, Q14, Q15, R17, R19, R21, R5
